File: asic_pwr.kicad_sch (KiCad schematic)
At the start: 39 parts, among them J9 Battery Terminals, U4 DA000001

Commit message: Minor corrections
Parts:
- FB1, FB3, L4, R4, TP1, TP13, TP17, TP23, TP6, TP7: value ~ -> (none)
