File: bt_soc.kicad_sch (KiCad schematic)
At the start: 28 parts, among them J6 GND_EDGE, J7 1V8_EDGE, J8 BT_ANT, U2 W25Q16JVBYIQ, U3 EM9305, Y1 48 MHz

Commit message: Minor corrections
Parts:
- removed U2: W25Q16JVBYIQ, LEGO:WLCSP-8_Winbond_BY, symbol LEGO:W25Q16JVBYIQ
- added U2: W25Q16JWBYIQ, LEGO:WLCSP-8_Winbond_BY, symbol LEGO:W25Q16JWBYIQ
- TP10, TP15, TP16, TP19, TP2, TP27, TP3, TP8, TP9: value ~ -> (none)
Connections:
- net +1V8: now also U2.A1 (VCC), U2.B1 (~{HOLD}/~{RESET}/IO_{3}), U2.C2 (~{WP}/IO_{2})
- net CS2: now also U2.A2 (~{CS})
- net GND: now also U2.D2 (GND)
- net MISO: now also U2.B2 (DO/IO_{1})
- net MOSI: now also U2.D1 (DI/IO_{0})
- net SCK: now also U2.C1 (CLK)
- net VIB_EN renamed ACEL_EN
- net VIB_INT renamed ACEL_INT
