File: lego_smart_brick.kicad_sch (KiCad schematic)
At the start: 0 parts

Commit message: Minor corrections
Other:
- sheet ASIC_SENSE ports: added ACEL_EN, ACEL_INT; removed VIB_EN, VIB_INT
- sheet BT_SOC ports: added ACEL_EN, ACEL_INT; removed VIB_EN, VIB_INT
Changed lines of the file:
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@@
 (kicad_sch
-	(version 20250114)
+	(version 20260306)
 	(generator "eeschema")
-	(generator_version "9.0")
+	(generator_version "10.0")
 	(paper "A4")
 	(rectangle
@@
 		)
 		(fill
-			(color 0 0 0 0.0000)
+			(color 0 0 0 0)
 		)
 		(property "Sheetname" "ASIC_PWR_NFC"
 			(at 149.86 71.6784 0)
+			(show_name no)
+			(do_not_autoplace no)
 			(effects
 				(font
@@
 		(property "Sheetfile" "asic_pwr.kicad_sch"
 			(at 149.86 83.7696 0)
+			(show_name no)
+			(do_not_autoplace no)
 			(effects
 				(font
@@
 		)
 		(fill
-			(color 0 0 0 0.0000)
+			(color 0 0 0 0)
 		)
 		(property "Sheetname" "BT_SOC"
 			(at 168.91 98.3484 0)
+			(show_name no)
+			(do_not_autoplace no)
 			(effects
 				(font
@@
 		(property "Sheetfile" "bt_soc.kicad_sch"
 			(at 168.91 120.5996 0)
+			(show_name no)
+			(do_not_autoplace no)
 			(effects
 				(font
@@
 			)
 		)
-		(pin "VIB_INT" output
-			(at 168.91 107.95 180)
+		(pin "GPIO4" bidirectional
+			(at 168.91 113.03 180)
 			(effects
 				(font
@@
 			)
 		)
-		(pin "VIB_EN" output
-			(at 168.91 110.49 180)
+		(pin "GPIO5" bidirectional
+			(at 168.91 115.57 180)
 			(effects
 				(font
@@
 			)
 		)
-		(pin "GPIO4" bidirectional
-			(at 168.91 113.03 180)
+		(pin "ACEL_INT" input
+			(at 168.91 107.95 180)
 			(effects
 				(font
@@
 			)
 		)
-		(pin "GPIO5" bidirectional
-			(at 168.91 115.57 180)
+		(pin "ACEL_EN" output
+			(at 168.91 110.49 180)
 			(effects
 				(font
@@
 		)
 		(fill
-			(color 0 0 0 0.0000)
+			(color 0 0 0 0)
 		)
 		(property "Sheetname" "ASIC_SENSE"
 			(at 132.08 98.3484 0)
+			(show_name no)
+			(do_not_autoplace no)
 			(effects
 				(font
@@
 		(property "Sheetfile" "asic.kicad_sch"
 			(at 132.08 120.5996 0)
+			(show_name no)
+			(do_not_autoplace no)
 			(effects
 				(font
@@
 			)
 		)
-		(pin "VIB_EN" input
-			(at 153.67 110.49 0)
+		(pin "GPIO4" bidirectional
+			(at 153.67 113.03 0)
 			(effects
 				(font
@@
 			)
 		)
-		(pin "GPIO4" bidirectional
-			(at 153.67 113.03 0)
+		(pin "GPIO5" bidirectional
+			(at 153.67 115.57 0)
 			(effects
 				(font
@@
 			)
 		)
-		(pin "GPIO5" bidirectional
-			(at 153.67 115.57 0)
+		(pin "ACEL_INT" output
+			(at 153.67 107.95 0)
 			(effects
 				(font
@@
 			)
 		)
-		(pin "VIB_INT" output
-			(at 153.67 107.95 0)
+		(pin "ACEL_EN" input
+			(at 153.67 110.49 0)
 			(effects
 				(font
