File: nfc.kicad_sch (KiCad schematic)
At the start: 60 parts, among them J1 NFC_ANT_RIGHT1, J10 NFC_LEFT1, J11 NFC_LEFT2, J12 NFC_ANT_FRONT2, J13 NFC_ANT_FRONT1, J14 NFC_ANT_BOTTOM1, J15 NFC_ANT_BOTTOM2, J16 NFC_ANT_BACK2, J2 NFC_ANT_RIGHT2, J3 NFC_ANT_TOP1, J4 NFC_ANT_TOP2, J5 NFC_ANT_BACK1

Commit message: Minor corrections
Parts:
- TP22, TP24, TP25, TP26, TP4, TP5: value ~ -> (none)
Other:
- note added: "Connected by copper coil"
